File: easyMySensors/easyMySens-v010.brd (EAGLE design)
At the start: 65 x 48 mm, 38 parts, among them IC1 ATSHA204A, IC2 REG1117, M1 ARDUINO-PRO-MINI-3.3V#NP, M2 NRF24L01+SMD, X1 1751277

Commit message: MySens easyProMini -Draft2
Parts:
- removed C5: (0.1uF), rcl:C1206
- removed JP12: (no value), pinhead-2:1X04-S
- added HM1, HM3, OPT: (no value), SparkFun-Connectors:1X04
- added HM2: (no value), SparkFun-Connectors:1X06
- added NMODULE: CONNECTOR_10DUPONT, TD-MySensors:DUPONT_10
- added X3: (no value), my:CON_350-103
- added X4: (no value), my:CON_350-103_O
- moved R3 32.2 mm to (16.5, 33.0), flipped to the bottom, turned to 180 degrees
- moved C2 31.4 mm to (44.5, 68.6), turned to 180 degrees
- moved C4 27.9 mm to (38.1, 68.6), turned to 180 degrees
- moved C10 24.8 mm to (23.5, 54.6), flipped to the bottom, turned to 0 degrees
- moved R2 23.9 mm to (38.1, 64.8), turned to 180 degrees
- moved U$3 23.1 mm to (57.4, 77.4), turned to 0 degrees
- moved C1 21.5 mm to (28.8, 34.6), flipped to the bottom, turned to 270 degrees
- moved R1 17.3 mm to (43.2, 64.8), turned to 180 degrees
- moved F1 16.5 mm to (42.8, 65.5), flipped to the bottom, turned to 0 degrees
- moved JP1 11.7 mm to (53.3, 54.6), turned to 90 degrees
- moved JP3 11.7 mm to (50.8, 54.6), turned to 90 degrees
- moved I2C-2 11.4 mm to (40.6, 49.0)
- moved MOTION 11.4 mm to (55.9, 54.6)
- moved REG1 1.91 mm to (41.4, 58.3)
- moved RS485 1.42 mm to (24.8, 49.5)
Connections:
- removed net CC_CS0: CC0.CSN
- removed net CC_IN_0: CC0.GDO2
- removed net CC_OUT_0: CC0.GDO0
- removed net MISO1: CC0.MISO
- removed net MOSI1: CC0.MOSI
- removed net SCK1: CC0.SCLK
- new net 1W_BUS: X3.B2, X4.B2
- new net 1W_GND: X3.B3, X4.B3
- new net 1W_VCC: X3.B1, X4.B1
- new net A3: HM2.2, M1.J6.5, NMODULE.3
- new net A6: M1.J3.2, OPT.4
- new net A7: M1.J3.3
- new net N$6: OPT.1
- net A0: now also HM1.3
- net A1: now also HM1.4, NMODULE.1
- net A2: now also HM2.1, NMODULE.2
- net A4: now also HM2.3, NMODULE.6
- net A5: now also HM2.4, NMODULE.7
- net ATSHA_D7: now also HM3.4
- net CSN: now also CC0.CSN
- net D3: now also HM2.5, NMODULE.4
- net D6: now also HM2.6
- net D9: now also HM3.3
- net GND: now also HM1.2, HM3.1, NMODULE.9, OPT.2; no longer C5.1
- net IRQ: now also CC0.GDO0, NMODULE.5
- net MISO: now also CC0.MISO
- net MOSI: now also CC0.MOSI
- net SCK: now also CC0.SCLK
- net UREG: now also HM1.1, NMODULE.10
- net VCC: now also HM3.2, NMODULE.8, OPT.3; no longer C5.2
Routing:
- net IRQ: track 65.4 -> 155.1 mm, vias 1 -> 5
- net A3: track 0.00 -> 58.5 mm, vias 0 -> 3
- net A2: track 0.00 -> 57.1 mm, vias 0 -> 3
- net ATSHA_D7: track 32.1 -> 83.9 mm, vias 1 -> 5
- net A1: track 23.1 -> 73.4 mm, vias 0 -> 4
- net D3: track 49.8 -> 90.9 mm, vias 0 -> 2
- net D9: track 6.80 -> 43.5 mm, vias 0 -> 2
- net A0: track 62.4 -> 94.9 mm, vias 1 -> 3
- net A5: track 135.7 -> 104.1 mm, vias 1 -> 5
- net D6: track 26.7 -> 57.9 mm, vias 0 -> 2
- net A4: track 127.3 -> 102.3 mm, vias 1 -> 2
- net A6: track 0.00 -> 18.1 mm, vias 0 -> 1
- net GND: track 324.6 -> 307.9 mm, vias 1 -> 3
- net 3.3V: track 76.0 -> 60.4 mm, vias 2 -> 4
- net SCK: track 34.4 -> 47.9 mm, vias 0 -> 1
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Other:
- outline, holes or cut-outs redrawn
- board text added: "HM"
- board text added: "uni versal"
