File: easyMySensors/easyMySens-v010.sch (EAGLE design)
At the start: 38 parts, among them IC1 ATSHA204A, IC2 REG1117, M1 ARDUINO-PRO-MINI-3.3V#NP, M2 NRF24L01+SMD, X1 1751277

Commit message: MySens easyProMini -Draft2
Parts:
- removed C5: (0.1uF), rcl:C-EUC1206
- removed JP12: (no value), pinhead-2:PINHD-1X04_2.54-S
- added HM1, HM3, OPT: (no value), SparkFun-Connectors:CONN_04
- added HM2: (no value), SparkFun-Connectors:CONN_06SILK_FEMALE_PTH
- added NMODULE: CONNECTOR_10DUPONT, TD-MySensors:CONNECTOR_10DUPONT
- added X3: (no value), my:CON_350-103
- added X4: (no value), my:CON_350-103OHNE_RAND
Connections:
- removed net CC_CS0: CC0.CSN
- removed net CC_IN_0: CC0.GDO2
- removed net CC_OUT_0: CC0.GDO0
- removed net MISO1: CC0.MISO
- removed net MOSI1: CC0.MOSI
- removed net SCK1: CC0.SCLK
- new net 1W_BUS: X3.B-2, X4.B-2
- new net 1W_GND: X3.B-3, X4.B-3
- new net 1W_VCC: X3.B-1, X4.B-1
- new net A3: HM2.2, M1.A3, NMODULE.3
- new net A6: M1.A6, OPT.4
- new net A7: M1.A7
- new net N$6: OPT.1
- net A0: now also HM1.3
- net A1: now also HM1.4, NMODULE.1
- net A2: now also HM2.1, NMODULE.2
- net A4: now also HM2.3, NMODULE.6
- net A5: now also HM2.4, NMODULE.7
- net ATSHA_D7: now also HM3.4
- net CSN: now also CC0.CSN
- net D3: now also HM2.5, NMODULE.4
- net D6: now also HM2.6
- net D9: now also HM3.3
- net GND: now also HM1.2, HM3.1, NMODULE.9, OPT.2; no longer C5.1
- net IRQ: now also CC0.GDO0, NMODULE.5
- net MISO: now also CC0.MISO
- net MOSI: now also CC0.MOSI
- net SCK: now also CC0.SCLK
- net UREG: now also HM1.1, NMODULE.10
- net VCC: now also HM3.2, NMODULE.8, OPT.3; no longer C5.2
Other:
- note added: "??? B1 ??"
- note added: "???Platzhalter für Klemmen ???"
- note added: "A3 für SHA Chip!"
- note added: "ATSHA204 authentication chip optional for MySensors"
- note added: "Achtung nur wenn physikalisch an der Position von GND.3 der A5 Pin ist verbinden !!!"
- note added: "Condensator at IC2..."
- note added: "Div"
- note added: "Ereiterungen zur HM-Universalplatine kommen auf die Rückseite der Platine"
- note added: "HomeMatic Universal (Pa-Pa)"
- note added: "MySX"
- note added: "RS485"
- note added: "Radios (nur eins erlaubt!)"
- note added: "Schraub 3,5mm"
- note added: "Terminierung mit Pull-Widerständen. Zwischen A und B 150 Ohm, von A 330 Ohm nach VCC, von B 330 Ohm nach GND. Damit wird er Bus auf HIGH gehalten wenn Teilnehmer passiv sind. AC-Widerstand ca. bei 120 Ohm (150 // (330+330)) = 122,2."
- note added: "easy MySensors-HM"
- note removed: "ATSHA204 authentication chip"
- note removed: "Achtung nur wenn an der Position von GND.3 der A5 Pin ist verbinden !!!"
- note removed: "Easy PCB - Rev 9"
- note removed: "Optional !"
- note removed: "Terminierung um Pull-Widerständen. Zwischen A und B 150 Ohm, von A 330 Ohm nach Vcc, von B 330 Ohm nach GND. Damit wird er Bus auf HIGH gehalten wenn alle Teilnehmer passiv sind. Der AC-Widerstand liegt ebenfalls ca. bei 120 Ohm (150 // (330+330)) = 122,2."
- moved on the sheet: A4, C10, C3, C6, CC0, F1, IC1, M2, MYSX, R3, R4, R5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
