File: MySensors-HM-easy-RFM-NRF-CC1101-RS485/easyMySens-v024.brd (EAGLE design)
At the start: 65 x 48 mm, 43 parts, among them IC1 ATSHA204A, IC2 REG1117, M1 ARDUINO-PRO-MINI-3.3V#NP, M2 NRF24L01+SMD, X1 1751277

Commit message: MySens V01 (ordered)
Parts:
- removed MYSX: (no value), pinhead-2:2X08
- removed R3: (no value), rcl:R0805
- removed RAW(MYSX): (no value), jumper:SJ
- removed X4: (no value), my:CON_350-103_O
- added A0, D7, I2C., UART: DIP Grove, con-lstb:MA04-1
- added ANT, ANT1: (no value), pinhead:1X01
- added C15, C27, C29: 10uF, Discrete-new:C0603
- added C16, C28, C30: 100nF, Discrete-new:C0603
- added RAW: (no value), jumper:SJ
- X1: value 1751277 -> 1751280; device con-phoenix-350:1751277 -> con-phoenix-350:1751280
- X3: value (none) -> 1751280; device my:CON_350-103 -> con-phoenix-350:1751280
- moved X3 27.9 mm to (11.0, 36.0), flipped to the bottom, turned to 180 degrees
- moved X1 5.53 mm to (11.0, 41.0)
- moved C3 3.62 mm to (31.1, 65.7), turned to 90 degrees
- moved A4 1.43 mm to (31.8, 49.5)
- moved RFM69W 0.90 mm to (26.0, 62.2)
- moved R4 0.76 mm to (14.7, 50.8)
- moved X2 0.67 mm to (0.00, 65.4)
- moved CC0 0.64 mm to (25.6, 77.0)
- moved X5 0.48 mm to (0.00, 70.5)
Connections:
- removed net 1W_BUS: X3.B2, X4.B2
- removed net 1W_GND: X3.B3, X4.B3
- removed net 1W_VCC: X3.B1, X4.B1
- removed net CE: M2.CE
- removed net N$1: MYSX.1, RAW(MYSX).2
- removed net N$3: RFM69W.RESET
- removed net N$6: OPT.1
- new net FREE: X1.1, X3.1
- new net RAW: M1.J6.1, RAW.1
- net 3.3V: no longer MYSX.2
- net A: now also X1.3, X3.3; no longer X1.2
- net A0: no longer MYSX.15
- net A1: now also A0.2; no longer MYSX.16
- net A2: now also A0.1
- net A4: now also I2C..2; no longer MYSX.14
- net A5: now also I2C..1; no longer MYSX.13
- net A7: now also OPT.1
- net ANT0: now also ANT.1
- net B: now also X1.4, X3.4; no longer X1.3
- net D3: no longer MYSX.9, R3.2
- net D5: now also D7.2; no longer MYSX.11
- net D6: now also D7.1; no longer MYSX.12
- net D9: now also M2.CE
- net GND: now also A0.4, C15.1, C16.1, C27.2, C28.2, C29.2, C30.2, D7.4, I2C..4, UART.4, X1.5, X3.5; no longer MYSX.4, MYSX.8, X1.4
- net IRQ: no longer MYSX.10
- net N$16: now also ANT1.1
- net RESET: no longer MYSX.7
- net RX: now also UART.1; no longer MYSX.6
- net TX: now also UART.2; no longer MYSX.5
- net UREG: now also RAW.2, X1.2, X3.2; no longer M1.J6.1, RAW(MYSX).1, X1.1
- net VCC: now also A0.3, C15.2, C16.2, C27.1, C28.1, C29.1, C30.1, D7.3, I2C..3, UART.3, X1.6, X3.6; no longer MYSX.3, R3.1, X1.5
Routing:
- net IRQ: track 155.1 -> 108.5 mm, vias 5 -> 3
- net UREG: track 181.0 -> 136.9 mm
- net RX: track 2.54 -> 44.2 mm
- net N$1: track 34.7 -> 0.00 mm, vias 1 -> 0
- net TX: track 7.88 -> 41.2 mm
- net D3: track 90.9 -> 61.3 mm, vias 2 -> 0
- net GND: track 307.9 -> 336.0 mm, vias 3 -> 19
- net A2: track 57.1 -> 79.8 mm
- net D5: track 14.6 -> 36.1 mm, vias 3 -> 0
- net A0: track 94.9 -> 75.9 mm, vias 3 -> 1
- net 3.3V: track 60.4 -> 48.4 mm, vias 4 -> 2
- net 1W_BUS: track 11.1 -> 0.00 mm
- net 1W_GND: track 11.1 -> 0.00 mm
- net 1W_VCC: track 11.1 -> 0.00 mm
- net D6: track 57.9 -> 68.3 mm, vias 2 -> 1
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- added copper zone on layer 1, net GND
- added copper zone on layer 16, net GND
Other:
- outline, holes or cut-outs redrawn
- board text added: "+"
- board text added: "-"
- board text added: "100nF"
- board text added: "150R"
- board text added: "1M"
- board text added: "22p"
- board text added: "330R"
- board text added: "470K"
- board text added: "A"
- board text added: "A1"
- board text added: "A2"
- board text added: "A4"
- board text added: "A5"
- board text added: "AMS1117"
- board text added: "ATSHA204A (MySensors optional)"
- board text added: "Analog"
- board text added: "Antenna"
- board text added: "B"
- board text added: "C1 10uF"
- board text added: "C2"
- board text added: "C3 10uF"
- board text added: "C4"
- board text added: "C6"
- board text added: "CC1101 for HM"
- board text added: "CE /D9"
- board text added: "CSN"
- board text added: "D4"
- board text added: "D5"
- board text added: "D6"
- board text added: "DIO0"
- board text added: "Digital"
- board text added: "Fuse1"
- board text added: "GND"
- board text added: "Grove Connectors"
- board text added: "IN"
- board text added: "IRQ"
- board text added: "MISO"
- board text added: "MOSI"
- board text added: "Max487"
- board text added: "Mini360"
- board text added: "NC"
- board text added: "NSS"
- board text added: "OUT"
- board text added: "Please include the cutouts..."
- board text added: "R1"
- board text added: "R2"
- board text added: "R4"
- board text added: "R5/6"
- board text added: "RST"
- board text added: "RX"
- board text added: "Reg1"
- board text added: "SCK"
- board text added: "SCL"
- board text added: "SDA"
- board text added: "TX"
- board text added: "UART"
- board text added: "UREG"
- board text added: "VCC"
- board text added: "uni- versal"
- board text removed: "4,7uF"
- board text removed: "A5/SCL SDA GND VCC"
- board text removed: "Checken"
- board text removed: "Gnd"
- board text removed: "MysX 2.4"
- board text removed: "VCC GND RAW"
- board text removed: "Vout"
- board text removed: "uni versal"
