File: MySensors-HM-easy-RFM-NRF-CC1101-RS485/easyMySens-v024.sch (EAGLE design)
At the start: 43 parts, among them IC1 ATSHA204A, IC2 REG1117, M1 ARDUINO-PRO-MINI-3.3V#NP, M2 NRF24L01+SMD, X1 1751277

Commit message: MySens V01 (ordered)
Parts:
- removed MYSX: (no value), pinhead-2:PINHD-2X08_2.54
- removed R3: (no value), rcl:R-EU_R0805
- removed RAW(MYSX): (no value), jumper:SJ
- removed X4: (no value), my:CON_350-103OHNE_RAND
- added A0, D7, I2C., UART: DIP Grove, con-lstb:MA04-1
- added ANT, ANT1: (no value), pinhead:PINHD-1X1
- added C15, C27, C29: 10uF, Discrete-new:CAP-0603
- added C16, C28, C30: 100nF, Discrete-new:CAP-0603
- added RAW: (no value), jumper:SJ
- X1: value 1751277 -> 1751280; device con-phoenix-350:1751277 -> con-phoenix-350:1751280
- X3: value (none) -> 1751280; device my:CON_350-103 -> con-phoenix-350:1751280
Connections:
- removed net 1W_BUS: X3.B-2, X4.B-2
- removed net 1W_GND: X3.B-3, X4.B-3
- removed net 1W_VCC: X3.B-1, X4.B-1
- removed net CE: M2.CE
- removed net N$1: MYSX.1, RAW(MYSX).2
- removed net N$3: RFM69W.RESET
- removed net N$6: OPT.1
- new net FREE: X1-1.K, X3-1.K
- new net RAW: M1.RAW, RAW.1
- net 3.3V: no longer MYSX.2
- net A: now also X1-3.K, X3-3.K; no longer X1-2.K
- net A0: no longer MYSX.15
- net A1: now also A0.2; no longer MYSX.16
- net A2: now also A0.1
- net A4: now also I2C..2; no longer MYSX.14
- net A5: now also I2C..1; no longer MYSX.13
- net A7: now also OPT.1
- net ANT0: now also ANT.1
- net B: now also X1-4.K, X3-4.K; no longer X1-3.K
- net D3: no longer MYSX.9, R3.2
- net D5: now also D7.2; no longer MYSX.11
- net D6: now also D7.1; no longer MYSX.12
- net D9: now also M2.CE
- net GND: now also A0.4, C15.1, C16.1, C27.2, C28.2, C29.2, C30.2, D7.4, I2C..4, UART.4, X1-5.K, X3-5.K; no longer MYSX.4, MYSX.8, X1-4.K
- net IRQ: no longer MYSX.10
- net N$16: now also ANT1.1
- net RESET: no longer MYSX.7
- net RX: now also UART.1; no longer MYSX.6
- net TX: now also UART.2; no longer MYSX.5
- net UREG: now also RAW.2, X1-2.K, X3-2.K; no longer M1.RAW, RAW(MYSX).1, X1-1.K
- net VCC: now also A0.3, C15.2, C16.2, C27.1, C28.1, C29.1, C30.1, D7.3, I2C..3, UART.3, X1-6.K, X3-6.K; no longer MYSX.3, R3.1, X1-5.K
Other:
- note removed: "???Platzhalter für Klemmen ???"
- note removed: "MySX"
- moved on the sheet: X1-1, X1-2, X1-3, X1-4, X1-5, X2
