File: MySensors-HM-easy-RFM-NRF-CC1101-RS485/MicroMySens-v003.sch (EAGLE design)
At the start: 52 parts, among them IC1 ATSHA204A, IC2 REG1117, M1 ARDUINO-PRO-MINI-3.3V#NP, M2 NRF24L01+SMD, X1 1751280, X3 1751280

Commit message: Some new easyBoards
Parts:
- removed A0, D7, I2C., UART: DIP Grove, con-lstb:MA04-1
- removed A4, ANT1: (no value), pinhead:PINHD-1X1
- removed BH1750, I2C-1, I2C-2, JP1, JP3, MOTION: (no value), pinhead-2:PINHD-1X04_2.54-S
- removed BOOST: R-78C1.8-1.0, dc-dc-converter:R-78C1.8-1.0
- removed C1: 10uF, rcl:C-EUC1210
- removed C10: 22p, rcl:C-EUC0805
- removed C16, C28, C30: 100nF, Discrete-new:CAP-0603
- removed C2: 0.1uF, rcl:C-EUC1206
- removed C27, C29: 10uF, Discrete-new:CAP-0603
- removed C3: 10uF, rcl:CPOL-EUSMCC
- removed C4: 0,1uF, rcl:C-EUC1206
- removed C6: 22pF, rcl:C-EUC0805
- removed CC0: CC1101, wireless:CC1101_MODULE1SMD
- removed F1: 1812L, ptc-littlefuse:1812L
- removed IC2: REG1117, burr-brown:REG1117
- removed M1: ARDUINO-PRO-MINI-3.3V#NP, diy-modules:ARDUINO-PRO-MINI-3.3V#NP
- removed M2: NRF24L01+SMD, wireless:NRF24L01+SMD
- removed NMODULE: CONNECTOR_10DUPONT, TD-MySensors:CONNECTOR_10DUPONT
- removed OPT: (no value), SparkFun-Connectors:CONN_04
- removed R1: 1M, rcl:R-EU_R0805
- removed R5, R6: 330R, rcl:R-EU_R0805
- removed RAW: (no value), jumper:SJ
- removed REG1: LP2950Z, linear:LP2950Z
- removed REG2: STEP-DWN-MP2307, diy-modules:DC-DC-STEP-DOWN-MP2307
- removed RFM69W: RFM69HW, hoperf:RFM69HW
- removed RS485: MAX487ECSA+, Maxim_By_element14_Batch_1:MAX487ECSA+
- removed U$3: 2.1MMJACKTHM, adafruit:2.1MMJACKTHM
- removed X1, X3: 1751280, con-phoenix-350:1751280
- removed X2, X5: (no value), adafruit:SMACONNECTOR_EDGE
- added C14: 30pf, doug:CAP0805
- added C31, C32: 100n, rcl:C-EUC0805
- added C5: 220uF, rcl:CPOL-EUE5-8.5
- added C7: (no value), rcl:C-EUC1812
- added IC31: ATMEGA168-TQFP, atmel:ATMEGA168-TQFP
- added R34: (no value), rcl:R-EU_R0805
- added U1: RFM69HCW, doug:RFM69HCW
- added X31: M03X2, mechanics:M03X2
- added Y2: 8MHZ, SparkFun-FreqCtrl:CRYSTALTXC-7A
- ANT: value (none) -> MICRO RF; device pinhead:PINHD-1X1 -> SparkFun-Connectors:M01PTH
- C15: value 10uF -> 30pf; device Discrete-new:CAP-0603 -> doug:CAP0805
- R2: value 470K -> 10k; device rcl:R-EU_R0805 -> doug:RESISTOR0805-RES
- R4: value 150R -> 1M; device rcl:R-EU_R0805 -> doug:RESISTOR0805-RES
Connections:
- removed net 3.3V: C3.+, IC1.VCC, M2.VCC, RFM69W.VCC
- removed net A: R4.1, R5.2, RS485.A, X1-3.K, X3-3.K
- removed net A6: M1.A6, OPT.4
- removed net A7: M1.A7, OPT.1
- removed net ANT0: ANT.1, CC0.ANT, X5.ANT
- removed net B: R4.2, R6.1, RS485.B, X1-4.K, X3-4.K
- removed net CSN: CC0.CSN, M1.D10, M2.CSN, RFM69W.NSS
- removed net D4: M1.D4, MOTION.3
- removed net D5: D7.2, M1.D5
- removed net D8: M1.D8, RS485.RO
- removed net FREE: X1-1.K, X3-1.K
- removed net IN: F1.2, U$3.TIP
- removed net IRQ: CC0.GDO0, M1.D2, M2.IRQ, NMODULE.5, RFM69W.DIO0, RS485.DE, RS485.~RE
- removed net MISO: CC0.MISO, M1.D12, M2.MISO, RFM69W.MISO
- removed net MOSI: CC0.MOSI, M1.D11, M2.MOSI, RFM69W.MOSI
- removed net RAW: M1.RAW, RAW.1
- removed net RESET: M1.RST.2
- removed net RX: M1.D0/RX, UART.1
- removed net SCK: CC0.SCLK, M1.D13, M2.SCK, RFM69W.SCK
- removed net TX: M1.D1/TX, UART.2
- new net ANT: ANT.1, U1.ANT
- new net CE-A: IC31.PB1(OC1A)
- new net D10_SS: IC31.PB2(SS/OC1B), R2.1, U1.NSS
- new net D11_MOSI: IC31.PB3(MOSI/OC2), U1.MOSI
- new net D12_MISO: IC31.PB4(MISO), U1.MISO
- new net D13_SCK: IC31.PB5(SCK), U1.SCK, X31.3
- new net D2_INT0: IC31.PD2(INT0), U1.DIO0
- new net D7-ATSHA: IC1.SDA, IC31.PD7(AIN1)
- new net M-RES: IC31.PC6(/RESET), R34.2, X31.5
- new net MISO-A: X31.1
- new net MOSI-A: X31.4
- new net N$13: C32.1, IC31.AREF
- new net N$14: U1.DIO2
- new net N$15: U1.DIO1
- new net N$19: C15.2, IC31.PB7(XTAL2/TOSC2), R4.1, Y2.1
- new net N$3: C14.2, IC31.PB6(XTAL1/TOSC1), R4.2, Y2.2
- new net RX1: IC31.PD1(TXD)
- new net TX1: IC31.PD0(RXD)
- net A0: no longer C4.2, M1.A0, R1.2, R2.2
- net A1: no longer A0.2, M1.A1, NMODULE.1
- net A2: no longer A0.1, M1.A2, NMODULE.2
- net A3: no longer M1.A3, NMODULE.3
- net A4: no longer A4.1, BH1750.3, I2C-1.3, I2C-2.3, I2C..2, M1.A4, NMODULE.6
- net A5: no longer BH1750.4, I2C-1.4, I2C-2.4, I2C..1, M1.A5, M1.GND.3, MOTION.4, NMODULE.7
- net ATSHA_D7: no longer IC1.SDA, M1.D7
- net D3: no longer M1.D3, NMODULE.4
- net D6: no longer D7.1, M1.D6
- net D9: no longer M1.D9, M2.CE, RS485.DI
- net GND: now also C14.1, C31.2, C32.2, C5.+, C7.2, IC31.AGND, IC31.GND@1, IC31.GND@2, U1.GND_1, U1.GND_2, U1.GND_3, X31.6; no longer A0.4, BH1750.2, BOOST.GND, C1.2, C10.1, C16.1, C2.2, C27.2, C28.2, C29.2, C3.-, C30.2, C4.1, C6.1, CC0.GND@1, CC0.GND@2, CC0.GND@3, D7.4, I2C-1.2, I2C-2.2, I2C..4, IC2.GND, JP1.1, JP1.2, JP1.3, JP1.4, M1.GND.1, M1.GND.2, M2.GND, MOTION.2, NMODULE.9, OPT.2, R2.1, R6.2, REG1.GND, REG2.IN-, REG2.OUT-, RFM69W.GNDA, RFM69W.GNDB, RS485.GND, U$3.RING, UART.4, X1-5.K, X2.GND1, X2.GND2, X2.GND3, X2.GND4, X3-5.K, X5.GND1, X5.GND2, X5.GND3, X5.GND4
- net N$16: now also U1.RESET; no longer ANT1.1, RFM69W.ANT, X2.ANT
- net UREG: no longer BOOST.VIN, C2.1, F1.1, IC2.VIN, NMODULE.10, R1.1, RAW.2, REG1.I, REG2.IN+, X1-2.K, X3-2.K
- net VCC: now also C31.1, C5.-, C7.1, IC1.VCC, IC31.AVCC, IC31.VCC@1, IC31.VCC@2, R2.2, R34.1, U1.3.3V, X31.2; no longer A0.3, BH1750.1, BOOST.VOUT, C1.1, C10.2, C15.2, C16.2, C27.1, C28.1, C29.1, C30.1, C6.2, CC0.VCC, D7.3, I2C-1.1, I2C-2.1, I2C..3, IC2.VOUT, JP3.1, JP3.2, JP3.3, JP3.4, M1.VCC, MOTION.1, NMODULE.8, OPT.3, R5.1, REG1.O, REG2.OUT+, RS485.VCC, UART.3, X1-6.K, X3-6.K
Other:
- note added: "ARM-Debugger"
- note added: "MEGA328"
- note added: "Nur ohne Homematic möglich"
- note added: "connect RES and GND"
- note added: "for flashing with bootloader"
- note added: "oscillator"
- note added: "use internal"
- note removed: "A3 für SHA Chip!"
- note removed: "ATSHA204 authentication chip optional for MySensors"
- note removed: "Achtung nur wenn physikalisch an der Position von GND.3 der A5 Pin ist verbinden !!!"
- note removed: "Arduino Pro Mini"
- note removed: "BMP280"
- note removed: "Condensator at IC2..."
- note removed: "Div"
- note removed: "Free Pins"
- note removed: "Motion"
- note removed: "Nrf24l01+ Radio"
- note removed: "Nur mit 3,3V Arduino!"
- note removed: "Power Converters"
- note removed: "RFM69(H)W"
- note removed: "RS485"
- note removed: "Radio 0"
- note removed: "Radios (nur eins erlaubt!)"
- note removed: "Schraub 3,5mm"
- note removed: "Terminierung mit Pull-Widerständen. Zwischen A und B 150 Ohm, von A 330 Ohm nach VCC, von B 330 Ohm nach GND. Damit wird er Bus auf HIGH gehalten wenn Teilnehmer passiv sind. AC-Widerstand ca. bei 120 Ohm (150 // (330+330)) = 122,2."
- note removed: "VDD-Config siehe 1Wire..."
- note removed: "because max. input voltage Vi = 5.25 V for NRF24L01+."
- note removed: "easy MySensors-HM"
- note removed: "no resistor divider for CE necessary,"
- moved on the sheet: HM1, HM2, HM3, IC1
