File: MySensors-HM-easy-RFM-NRF-CC1101-RS485/easyMySens-v030.sch (EAGLE design)
At the start: 33 parts, among them IC31 ATSHA204A, M31 NRF24L01+SMD, X7 1751264

Commit message: Some new easyBoards
Parts:
- removed C9: 220p, rcl:C-EUC0805
- removed IC31: ATSHA204A, Sensor:ATSHA204A
- removed IRQ, RAW(MYSX), V: (no value), jumper:SJ
- removed JP10, JP2, JP4, JP6: (no value), pinhead-2:PINHD-1X04_2.54-S
- removed JP19: (no value), pinhead:PINHD-1X2
- removed M31: NRF24L01+SMD, wireless:NRF24L01+SMD
- removed MAX487: MAX481CPA, maxim-4:MAX481CPA
- removed MCU2: ARDUINO_PRO_MICRO_NO_A0-A1, arduino:ARDUINO_PRO_MICRO_NO_A0-A1
- removed MYSX: (no value), pinhead-2:PINHD-2X08_2.54
- removed NRF24L01+: WIRELESS-NRF24L01, diy-modules:WIRELESS-NRF24L01
- removed PRO-MINI: ARDUINO_PRO_MINI_NO_A0-A1, arduino:ARDUINO_PRO_MINI_NO_A0-A1
- removed U$2: NANO, Arduino-clone:NANO
- removed X7: 1751264, con-phoenix-350:1751264
- added A0, D7, I2C., UART: DIP Grove, con-lstb:MA04-1
- added A4, ANT, ANT1: (no value), pinhead:PINHD-1X1
- added BH1750, I2C-1, I2C-2, JP1, JP3, MOTION: (no value), pinhead-2:PINHD-1X04_2.54-S
- added C15, C27, C29: 10uF, Discrete-new:CAP-0603
- added C16, C28, C30: 100nF, Discrete-new:CAP-0603
- added C6: 22pF, rcl:C-EUC0805
- added CC0: CC1101, wireless:CC1101_MODULE1SMD
- added F1: 1812L, ptc-littlefuse:1812L
- added HM1, HM3, OPT: (no value), SparkFun-Connectors:CONN_04
- added HM2: (no value), SparkFun-Connectors:CONN_06SILK_FEMALE_PTH
- added IC1: ATSHA204A, Sensor:ATSHA204A
- added IC2: REG1117, burr-brown:REG1117
- added ICLUSION: DTSM-3, mechanics:DTSM-3
- added L1: 4,7uH, SparkFun-Passives:INDUCTOR0805
- added M1: ARDUINO-PRO-MINI-3.3V#NP, diy-modules:ARDUINO-PRO-MINI-3.3V#NP
- added M2: NRF24L01+SMD, wireless:NRF24L01+SMD
- added NMODULE: CONNECTOR_10DUPONT, TD-MySensors:CONNECTOR_10DUPONT
- added R6: 330R, rcl:R-EU_R0805
- added R7: 10K, rcl:R-EU_R0805
- added RAW: (no value), jumper:SJ
- added RFM69W: RFM69HW, hoperf:RFM69HW
- added STEPUP: TLV61224, TLV61224:TI-TLV61224
- added X1, X3: 1751280, con-phoenix-350:1751280
- added X2, X5: (no value), adafruit:SMACONNECTOR_EDGE
- C3: value 4,7 -> 10uF
- C5: value (0.1uF) -> 10uF; device rcl:C-EUC1206 -> SparkFun-Passives:CAP0805
- R3: value (none) -> 10K
- R4: value 60 -> 150R
- R5: value 60 -> 330R
Connections:
- removed net +3V3: IC31.VCC
- removed net 3V3: U$2.3.3V
- removed net BOOSTIN: BOOST.VIN, JP2.4, R1.1
- removed net BOOSTOUT: BOOST.VOUT, C5.2, JP4.4
- removed net CE: M31.CE, NRF24L01+.CE
- removed net CE_D9: MCU2.D9, PRO-MINI.D9
- removed net C_EEP_5: MCU2.D8, PRO-MINI.D8
- removed net D7: U$2.D7
- removed net GDO0_D3: MCU2.D3, PRO-MINI.D3
- removed net GDO2_D2: MCU2.D2, PRO-MINI.D2
- removed net LED_ERR_D4: MCU2.D4, PRO-MINI.D4
- removed net LED_RX_D6: MCU2.D6, PRO-MINI.D6
- removed net LED_TX_D5: MCU2.D5, PRO-MINI.D5
- removed net N$1: MYSX.1, RAW(MYSX).2
- removed net N$2: U$2.5.5V, V.1
- removed net N$20: U$2.AREF
- removed net N$21: C9.1, R4.1, R5.1
- removed net N$24: U$2.A2
- removed net N$25: U$2.A3
- removed net N$26: U$2.A4
- removed net N$27: U$2.A5
- removed net N$28: U$2.A6
- removed net N$29: U$2.A7
- removed net N$3: IRQ.2, U$2.D2
- removed net N$31: U$2.RST
- removed net R1IN: C2.1, JP2.1, REG1.I
- removed net R1OUT: C1.1, JP4.1, REG1.O
- removed net R2IN: JP2.2, REG2.IN+
- removed net R2OUT: JP4.2, REG2.OUT+
- new net A2: A0.1, HM2.1, M1.A2, NMODULE.2
- new net A3: HM2.2, M1.A3, NMODULE.3
- new net A6: M1.A6, OPT.4
- new net A7: M1.A7, OPT.1
- new net ANT0: ANT.1, CC0.ANT, X5.ANT
- new net IN: F1.2, X1-1.K, X3-1.K
- new net N$13: L1.2, STEPUP.SW
- new net N$16: ANT1.1, RFM69W.ANT, X2.ANT
- new net VIN: C5.1, L1.1, STEPUP.EN, STEPUP.VBAT
- net 3.3V: now also IC1.VCC, M2.VCC, RFM69W.VCC; no longer C3.+, M31.VCC, MYSX.2, NRF24L01+.VCC, V.2
- net A: now also R4.1, X1-3.K, X3-3.K; no longer MAX487G$1.A, X7-2.K
- net A0: now also HM1.3, M1.A0; no longer MYSX.15, U$2.A0
- net A1: now also A0.2, HM1.4, M1.A1, NMODULE.1; no longer MYSX.16, U$2.A1
- net A4: now also A4.1, BH1750.3, HM2.3, I2C-1.3, I2C-2.3, I2C..2, M1.A4, NMODULE.6, R3.2; no longer JP10.4, JP6.4, MYSX.14
- net A5: now also BH1750.4, HM2.4, I2C-1.4, I2C-2.4, I2C..1, M1.A5, M1.GND.3, MOTION.4, NMODULE.7, R7.2; no longer JP10.3, JP6.3, MYSX.13
- net ATSHA_D7: now also HM3.4, IC1.SDA, M1.D7; no longer IC31.SDA, MCU2.D7, PRO-MINI.D7
- net B: now also R6.1, X1-4.K, X3-4.K; no longer MAX487G$1.B, X7-3.K
- net CSN: now also CC0.CSN, M1.D10, M2.CSN, RFM69W.NSS; no longer M31.CSN, MCU2.D10, NRF24L01+.CSN, PRO-MINI.D10, U$2.D10
- net D3: now also HM2.5, M1.D3, NMODULE.4; no longer MYSX.9, R3.2, U$2.D3
- net D4: now also M1.D4, MOTION.3; no longer U$2.D4
- net D5: now also D7.2, M1.D5; no longer MYSX.11, U$2.D5
- net D6: now also D7.1, HM2.6, M1.D6; no longer MYSX.12, U$2.D6
- net D8: now also ICLUSION.2, M1.D8; no longer MAX487G$1.RO, U$2.D8
- net D9: now also HM3.3, M1.D9, M2.CE; no longer MAX487G$1.DI, U$2.D9
- net GND: now also A0.4, BH1750.2, C15.1, C16.1, C27.2, C28.2, C29.2, C30.2, C5.2, C6.1, CC0.GND@1, CC0.GND@2, CC0.GND@3, D7.4, HM1.2, HM3.1, I2C-1.2, I2C-2.2, I2C..4, IC1.GND, IC2.GND, ICLUSION.1, JP1.1, JP1.2, JP1.3, JP1.4, M1.GND.1, M1.GND.2, M2.GND, MOTION.2, NMODULE.9, OPT.2, R6.2, RFM69W.GNDA, RFM69W.GNDB, STEPUP.GND, UART.4, X1-5.K, X2.GND1, X2.GND2, X2.GND3, X2.GND4, X3-5.K, X5.GND1, X5.GND2, X5.GND3, X5.GND4; no longer C5.1, C9.2, IC31.GND, JP10.2, JP19.1, JP6.2, M31.GND, MCU2.GND@1, MCU2.GND@2, MYSX.4, MYSX.8, NRF24L01+.GND, PRO-MINI.GND@0, PRO-MINI.GND@1, U$2.GND, U$2.GND2, X7-4.K
- net IRQ: now also CC0.GDO0, M1.D2, M2.IRQ, NMODULE.5, RFM69W.DIO0; no longer IRQ.1, M31.IRQ, MAX487G$1.DE, MAX487G$1.RE/, MYSX.10, NRF24L01+.IRQ
- net MISO: now also CC0.MISO, M1.D12, M2.MISO, RFM69W.MISO; no longer M31.MISO, MCU2.D12/MISO, NRF24L01+.MISO, PRO-MINI.D12/MISO, U$2.D12
- net MOSI: now also CC0.MOSI, M1.D11, M2.MOSI, RFM69W.MOSI; no longer M31.MOSI, MCU2.D11/MOSI, NRF24L01+.MOSI, PRO-MINI.D11/MOSI, U$2.D11
- net RAW: now also M1.RAW, RAW.1; no longer JP4.3, U$2.RAW
- net RESET: now also M1.RST.2; no longer MYSX.7, U$2.RST1
- net RX: now also M1.D0/RX, UART.1; no longer MYSX.6, U$2.RX1
- net SCK: now also CC0.SCLK, M1.D13, M2.SCK, RFM69W.SCK; no longer M31.SCK, MCU2.D13/SCK, NRF24L01+.SCK, PRO-MINI.D13/SCK, U$2.D13
- net TX: now also M1.D1/TX, UART.2; no longer MYSX.5, U$2.TX0
- net UREG: now also BOOST.VIN, C2.1, F1.1, HM1.1, IC2.VIN, NMODULE.10, R1.1, RAW.2, REG1.I, REG2.IN+, X1-2.K, X3-2.K; no longer JP2.3, RAW(MYSX).1, X7-1.K
- net VCC: now also A0.3, BH1750.1, BOOST.VOUT, C1.1, C15.2, C16.2, C27.1, C28.1, C29.1, C3.+, C30.1, C6.2, CC0.VCC, D7.3, HM3.2, I2C-1.1, I2C-2.1, I2C..3, IC2.VOUT, JP3.1, JP3.2, JP3.3, JP3.4, M1.VCC, MOTION.1, NMODULE.8, OPT.3, R5.1, R7.1, REG1.O, REG2.OUT+, STEPUP.FB, STEPUP.VOUT, UART.3, X1-6.K, X3-6.K; no longer JP10.1, JP19.2, JP6.1, MYSX.3
Other:
- note added: "??? B1 ??"
- note added: "A3 für SHA Chip!"
- note added: "ATSHA204 authentication chip optional for MySensors"
- note added: "Achtung nur wenn physikalisch an der Position von GND.3 der A5 Pin ist verbinden !!!"
- note added: "Arduino Pro Mini"
- note added: "BMP280"
- note added: "Condensator at IC2..."
- note added: "Div"
- note added: "Ereiterungen zur HM-Universalplatine kommen auf die Rückseite der Platine"
- note added: "Grove (in "wrong" = normal 2,54mm size...)"
- note added: "HomeMatic Universal (Pa-Pa)"
- note added: "Motion"
- note added: "Neu in V1.0 -Pullups for IC2 possible -3V3 connected to VCC -Beschriftung "I2C" gefixt -Stepup integrated"
- note added: "Nur mit 3,3V Arduino!"
- note added: "RFM69(H)W"
- note added: "RS485"
- note added: "Radio 0"
- note added: "Radios (nur eins erlaubt!)"
- note added: "Schraub 3,5mm"
- note added: "Terminierung mit Pull-Widerständen. Zwischen A und B 150 Ohm, von A 330 Ohm nach VCC, von B 330 Ohm nach GND. Damit wird er Bus auf HIGH gehalten wenn Teilnehmer passiv sind. AC-Widerstand ca. bei 120 Ohm (150 // (330+330)) = 122,2."
- note added: "easy MySensors-HM"
- note added: "inclusion"
- note removed: "3.3 V/8 MHz version only!"
- note removed: "ATSHA204 authentication chip"
- note removed: "Easy PCB - Rev 9"
- note removed: "Optional !"
- note removed: "USB/serial converter is needed (3.3V!)"
- note removed: "to be connected to VCC, GND, TX and RX"
- moved on the sheet: BOOST, C1, C10, C2, C3, C4, C5, R1, R2, R3, R4, R5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
