File: MySensors-HM-easy-RFM-NRF-CC1101-RS485/easyMySens-v031.brd (EAGLE design)
At the start: 65 x 48 mm, 57 parts, among them IC1 ATSHA204A, IC2 REG1117, M1 ARDUINO-PRO-MINI-3.3V#NP, M2 NRF24L01+SMD, X1 1751280, X3 1751280

Commit message: little fixes for new easyBoards
Connections:
- net A4: now also BH1750.4, I2C-1.4, I2C-2.4; no longer BH1750.3, I2C-1.3, I2C-2.3
- net A5: now also BH1750.3, I2C-1.3, I2C-2.3; no longer BH1750.4, I2C-1.4, I2C-2.4
Routing:
- net A4: track 126.6 -> 119.5 mm
- net A5: track 123.7 -> 128.6 mm
- net GND: track 338.9 -> 341.2 mm
Other:
- board text added: "VCC GND SCL A4/SDA"
- board text removed: "VCC GND A4/SDA SCL"
