File: MySensors-HM-easy-RFM-NRF-CC1101-RS485/easyMySens-v031.sch (EAGLE design)
At the start: 57 parts, among them IC1 ATSHA204A, IC2 REG1117, M1 ARDUINO-PRO-MINI-3.3V#NP, M2 NRF24L01+SMD, X1 1751280, X3 1751280

Commit message: little fixes for new easyBoards
Connections:
- net A4: now also BH1750.4, I2C-1.4, I2C-2.4; no longer BH1750.3, I2C-1.3, I2C-2.3
- net A5: now also BH1750.3, I2C-1.3, I2C-2.3; no longer BH1750.4, I2C-1.4, I2C-2.4
Changed lines of the file:
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@@
-</segment>
-<segment>
-<pinref part="BH1750" gate="A" pin="3"/>
-<wire x1="116.84" y1="-40.64" x2="116.84" y2="-54.61" width="0.1524" layer="91"/>
-<label x="116.84" y="-54.61" size="1.778" layer="95" rot="R270" xref="yes"/>
-</segment>
-<segment>
-<pinref part="I2C-1" gate="A" pin="3"/>
-<wire x1="96.52" y1="-40.64" x2="96.52" y2="-54.61" width="0.1524" layer="91"/>
-<label x="96.52" y="-54.61" size="1.778" layer="95" rot="R270" xref="yes"/>
-</segment>
-<segment>
-<pinref part="I2C-2" gate="A" pin="3"/>
-<wire x1="91.44" y1="-12.7" x2="91.44" y2="-26.67" width="0.1524" layer="91"/>
-<label x="91.44" y="-26.67" size="1.778" layer="95" rot="R270" xref="yes"/>
 </segment>
 <segment>
@@
 <label x="-6.35" y="-43.18" size="1.27" layer="95" ratio="10"/>
 </segment>
+<segment>
+<pinref part="I2C-1" gate="A" pin="4"/>
+<wire x1="99.06" y1="-40.64" x2="99.06" y2="-48.26" width="0.1524" layer="91"/>
+<label x="99.06" y="-48.26" size="1.778" layer="95" rot="R270" xref="yes"/>
+</segment>
+<segment>
+<pinref part="BH1750" gate="A" pin="4"/>
+<wire x1="119.38" y1="-40.64" x2="119.38" y2="-48.26" width="0.1524" layer="91"/>
+<label x="119.38" y="-48.26" size="1.778" layer="95" rot="R270" xref="yes"/>
+</segment>
+<segment>
+<pinref part="I2C-2" gate="A" pin="4"/>
+<wire x1="93.98" y1="-12.7" x2="93.98" y2="-20.32" width="0.1524" layer="91"/>
+<label x="93.98" y="-20.32" size="1.778" layer="95" rot="R270" xref="yes"/>
+</segment>
 </net>
 <net name="A5" class="0">
@@
 <wire x1="-43.18" y1="205.74" x2="-55.88" y2="205.74" width="0.1524" layer="91"/>
 <label x="-55.88" y="205.74" size="1.778" layer="95" rot="R180" xref="yes"/>
-</segment>
-<segment>
-<pinref part="BH1750" gate="A" pin="4"/>
-<wire x1="119.38" y1="-40.64" x2="119.38" y2="-48.26" width="0.1524" layer="91"/>
-<label x="119.38" y="-48.26" size="1.778" layer="95" rot="R270" xref="yes"/>
-</segment>
-<segment>
-<pinref part="I2C-1" gate="A" pin="4"/>
-<wire x1="99.06" y1="-40.64" x2="99.06" y2="-48.26" width="0.1524" layer="91"/>
-<label x="99.06" y="-48.26" size="1.778" layer="95" rot="R270" xref="yes"/>
-</segment>
-<segment>
-<pinref part="I2C-2" gate="A" pin="4"/>
-<wire x1="93.98" y1="-12.7" x2="93.98" y2="-20.32" width="0.1524" layer="91"/>
-<label x="93.98" y="-20.32" size="1.778" layer="95" rot="R270" xref="yes"/>
 </segment>
 <segment>
@@
 <label x="-6.35" y="-45.72" size="1.27" layer="95" ratio="10"/>
 </segment>
+<segment>
+<pinref part="BH1750" gate="A" pin="3"/>
+<wire x1="116.84" y1="-40.64" x2="116.84" y2="-54.61" width="0.1524" layer="91"/>
+<label x="116.84" y="-54.61" size="1.778" layer="95" rot="R270" xref="yes"/>
+</segment>
+<segment>
+<pinref part="I2C-1" gate="A" pin="3"/>
+<wire x1="96.52" y1="-40.64" x2="96.52" y2="-54.61" width="0.1524" layer="91"/>
+<label x="96.52" y="-54.61" size="1.778" layer="95" rot="R270" xref="yes"/>
+</segment>
+<segment>
+<pinref part="I2C-2" gate="A" pin="3"/>
+<wire x1="91.44" y1="-12.7" x2="91.44" y2="-26.67" width="0.1524" layer="91"/>
+<label x="91.44" y="-26.67" size="1.778" layer="95" rot="R270" xref="yes"/>
+</segment>
 </net>
