File: MySens-GW-RS485-Nano/MySens-GWeasyRS485-Nano-V10-004.sch (EAGLE design)
At the start: 43 parts, among them X7 1751264

Commit message: Some new easyBoards
Parts:
- removed C3: 4,7, rcl:CPOL-EUSMCC
- removed JP17, JP18, JP2, JP4, JP5, JP7, JP9: (no value), pinhead-2:PINHD-1X04_2.54-S
- removed NRF24L01+: WIRELESS-NRF24L01, diy-modules:WIRELESS-NRF24L01
- added ANT1: (no value), pinhead:PINHD-1X1
- added IC1: ATSHA204A, Sensor:ATSHA204A
- added RFM69W: RFM69HW, hoperf:RFM69HW
- added X2: (no value), adafruit:SMACONNECTOR_EDGE
Connections:
- removed net BOOSTIN: BOOST.VIN, JP2.4, R1.1
- removed net BOOSTOUT: BOOST.VOUT, C5.2, JP4.4
- removed net CE: NRF24L01+.CE
- removed net N$1: MYSX.1, RAW(MYSX).2
- removed net R1IN: C2.1, JP2.1, REG1.I
- removed net R1OUT: C1.1, JP4.1, REG1.O
- removed net R2IN: JP2.2, REG2.IN+
- removed net R2OUT: JP4.2, REG2.OUT+
- removed net RAW: JP4.3, U$2.RAW
- removed net REG: REGULATED-1.KL
- removed net UREG: F1.1, JP2.3, RAW(MYSX).1, X7-1.K
- new net IN: BOOST.VIN, C2.1, F1.1, R1.1, RAW(MYSX).1, REG1.I, REG2.IN+, X7-1.K
- new net N$16: ANT1.1, RFM69W.ANT, X2.ANT
- new net OUT: BOOST.VOUT, C1.1, C5.2, REG1.O, REG2.OUT+, REGULATED-1.KL
- new net RW: MYSX.1, RAW(MYSX).2, U$2.RAW
- net 3.3V: now also IC1.VCC; no longer C3.+, NRF24L01+.VCC
- net 3V3: now also RFM69W.VCC
- net CSN: now also RFM69W.NSS; no longer NRF24L01+.CSN
- net D7: now also IC1.SDA
- net GND: now also IC1.GND, RFM69W.GNDA, RFM69W.GNDB, X2.GND1, X2.GND2, X2.GND3, X2.GND4; no longer C3.-, NRF24L01+.GND
- net IRQ: now also RFM69W.DIO0; no longer NRF24L01+.IRQ
- net MISO: now also RFM69W.MISO; no longer NRF24L01+.MISO
- net MOSI: now also RFM69W.MOSI; no longer NRF24L01+.MOSI
- net SCK: now also RFM69W.SCK; no longer NRF24L01+.SCK
Other:
- note added: "ATSHA204 authentication chip optional for MySensors"
- note added: "Nur mit 3,3V Arduino!"
- note added: "RFM69(H)W"
- note added: "Radios (nur eins erlaubt!)"
