File: RS485-Termination-Brasletti/Terminierung_RS485-006.sch (EAGLE design)
At the start: 9 parts, among them IC1 REG1117, X1 1751264

Commit message: Rs485 Term
Parts:
- added PAD1, PAD2, PAD3, PAD4: WIREPADSMD1,27-254, wirepad:WIREPADSMD1,27-254
Connections:
- removed net N$3: C3.1, R1.1, R2.2, R4.2, X1-3.K
- removed net N$4: C3.2, R2.1, R3.2, R4.1, X1-2.K
- new net A: C3.2, PAD2.P, R2.1, R3.2, R4.1, X1-2.K
- new net B: C3.1, PAD3.P, R1.1, R2.2, R4.2, X1-3.K
- net GND: now also PAD4.P
- net VCC: now also PAD1.P
Changed lines of the file:
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@@
 <part name="R4" library="resistor" deviceset="R-EU_" device="M1206"/>
 <part name="C3" library="resistor" deviceset="C-EU" device="C0805K" value="22pF"/>
+<part name="PAD1" library="wirepad" deviceset="WIREPAD" device="SMD1,27-254"/>
+<part name="PAD2" library="wirepad" deviceset="WIREPAD" device="SMD1,27-254"/>
+<part name="PAD3" library="wirepad" deviceset="WIREPAD" device="SMD1,27-254"/>
+<part name="PAD4" library="wirepad" deviceset="WIREPAD" device="SMD1,27-254"/>
 </parts>
 <sheets>
@@
 <instance part="R4" gate="G$1" x="2.54" y="-2.54" rot="R90"/>
 <instance part="C3" gate="G$1" x="10.16" y="-2.54"/>
+<instance part="PAD1" gate="G$1" x="-109.22" y="-12.7"/>
+<instance part="PAD2" gate="G$1" x="-109.22" y="-5.08"/>
+<instance part="PAD3" gate="G$1" x="-109.22" y="2.54"/>
+<instance part="PAD4" gate="G$1" x="-109.22" y="10.16"/>
 </instances>
 <busses>
@@
 <wire x1="-66.04" y1="22.86" x2="-66.04" y2="10.16" width="0.1524" layer="91"/>
 <junction x="-66.04" y="10.16"/>
+<pinref part="PAD4" gate="G$1" pin="P"/>
+<wire x1="-71.12" y1="10.16" x2="-106.68" y2="10.16" width="0.1524" layer="91"/>
+<junction x="-71.12" y="10.16"/>
 </segment>
 </net>
-<net name="N$3" class="0">
+<net name="B" class="0">
 <segment>
 <pinref part="X1" gate="-3" pin="K"/>
@@
 <wire x1="10.16" y1="2.54" x2="10.16" y2="0" width="0.1524" layer="91"/>
 <junction x="2.54" y="2.54"/>
+<pinref part="PAD3" gate="G$1" pin="P"/>
+<wire x1="-71.12" y1="2.54" x2="-106.68" y2="2.54" width="0.1524" layer="91"/>
+<junction x="-71.12" y="2.54"/>
+<label x="-68.58" y="2.54" size="1.778" layer="95"/>
 </segment>
 </net>
-<net name="N$4" class="0">
+<net name="A" class="0">
 <segment>
 <pinref part="X1" gate="-2" pin="K"/>
@@
 <junction x="2.54" y="-7.62"/>
 <wire x1="2.54" y1="-7.62" x2="-7.62" y2="-7.62" width="0.1524" layer="91"/>
+<pinref part="PAD2" gate="G$1" pin="P"/>
+<wire x1="-71.12" y1="-5.08" x2="-106.68" y2="-5.08" width="0.1524" layer="91"/>
+<junction x="-71.12" y="-5.08"/>
+<label x="-68.58" y="-5.08" size="1.778" layer="95"/>
 </segment>
 </net>
@@
 <junction x="-71.12" y="-12.7"/>
 <junction x="-60.96" y="-12.7"/>
+<pinref part="PAD1" gate="G$1" pin="P"/>
+<wire x1="-71.12" y1="-12.7" x2="-106.68" y2="-12.7" width="0.1524" layer="91"/>
 </segment>
 </net>
