File: RS485-Termination-Brasletti/Terminierung_RS485-007.brd (EAGLE design)
At the start: 14 x 23 mm, 13 parts, among them IC1 REG1117, X1 1751264

Commit message: rs485  Terminator update
Other:
- board size 14 x 23 mm -> 14 x 21 mm
- board text added: "1117"
Changed lines of the file:
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@@
 <layer number="19" name="Unrouted" color="6" fill="1" visible="yes" active="yes"/>
 <layer number="20" name="Dimension" color="24" fill="1" visible="yes" active="yes"/>
-<layer number="21" name="tPlace" color="7" fill="1" visible="no" active="yes"/>
+<layer number="21" name="tPlace" color="7" fill="1" visible="yes" active="yes"/>
 <layer number="22" name="bPlace" color="7" fill="1" visible="yes" active="yes"/>
-<layer number="23" name="tOrigins" color="15" fill="1" visible="no" active="yes"/>
+<layer number="23" name="tOrigins" color="15" fill="1" visible="yes" active="yes"/>
 <layer number="24" name="bOrigins" color="15" fill="1" visible="yes" active="yes"/>
-<layer number="25" name="tNames" color="7" fill="1" visible="no" active="yes"/>
+<layer number="25" name="tNames" color="7" fill="1" visible="yes" active="yes"/>
 <layer number="26" name="bNames" color="7" fill="1" visible="yes" active="yes"/>
-<layer number="27" name="tValues" color="7" fill="1" visible="no" active="yes"/>
+<layer number="27" name="tValues" color="7" fill="1" visible="yes" active="yes"/>
 <layer number="28" name="bValues" color="7" fill="1" visible="yes" active="yes"/>
-<layer number="29" name="tStop" color="7" fill="3" visible="no" active="yes"/>
-<layer number="30" name="bStop" color="7" fill="6" visible="no" active="yes"/>
-<layer number="31" name="tCream" color="7" fill="4" visible="no" active="yes"/>
-<layer number="32" name="bCream" color="7" fill="5" visible="no" active="yes"/>
-<layer number="33" name="tFinish" color="6" fill="3" visible="no" active="yes"/>
-<layer number="34" name="bFinish" color="6" fill="6" visible="no" active="yes"/>
-<layer number="35" name="tGlue" color="7" fill="4" visible="no" active="yes"/>
-<layer number="36" name="bGlue" color="7" fill="5" visible="no" active="yes"/>
-<layer number="37" name="tTest" color="7" fill="1" visible="no" active="yes"/>
-<layer number="38" name="bTest" color="7" fill="1" visible="no" active="yes"/>
-<layer number="39" name="tKeepout" color="4" fill="11" visible="no" active="yes"/>
-<layer number="40" name="bKeepout" color="1" fill="11" visible="no" active="yes"/>
-<layer number="41" name="tRestrict" color="4" fill="10" visible="no" active="yes"/>
-<layer number="42" name="bRestrict" color="1" fill="10" visible="no" active="yes"/>
-<layer number="43" name="vRestrict" color="2" fill="10" visible="no" active="yes"/>
-<layer number="44" name="Drills" color="7" fill="1" visible="no" active="yes"/>
-<layer number="45" name="Holes" color="7" fill="1" visible="no" active="yes"/>
-<layer number="46" name="Milling" color="3" fill="1" visible="no" active="yes"/>
-<layer number="47" name="Measures" color="7" fill="1" visible="no" active="yes"/>
-<layer number="48" name="Document" color="7" fill="1" visible="no" active="yes"/>
-<layer number="49" name="Reference" color="7" fill="1" visible="no" active="yes"/>
-<layer number="51" name="tDocu" color="7" fill="1" visible="no" active="yes"/>
-<layer number="52" name="bDocu" color="7" fill="1" visible="no" active="yes"/>
+<layer number="29" name="tStop" color="7" fill="3" visible="yes" active="yes"/>
+<layer number="30" name="bStop" color="7" fill="6" visible="yes" active="yes"/>
+<layer number="31" name="tCream" color="7" fill="4" visible="yes" active="yes"/>
+<layer number="32" name="bCream" color="7" fill="5" visible="yes" active="yes"/>
+<layer number="33" name="tFinish" color="6" fill="3" visible="yes" active="yes"/>
+<layer number="34" name="bFinish" color="6" fill="6" visible="yes" active="yes"/>
+<layer number="35" name="tGlue" color="7" fill="4" visible="yes" active="yes"/>
+<layer number="36" name="bGlue" color="7" fill="5" visible="yes" active="yes"/>
+<layer number="37" name="tTest" color="7" fill="1" visible="yes" active="yes"/>
+<layer number="38" name="bTest" color="7" fill="1" visible="yes" active="yes"/>
+<layer number="39" name="tKeepout" color="4" fill="11" visible="yes" active="yes"/>
+<layer number="40" name="bKeepout" color="1" fill="11" visible="yes" active="yes"/>
+<layer number="41" name="tRestrict" color="4" fill="10" visible="yes" active="yes"/>
+<layer number="42" name="bRestrict" color="1" fill="10" visible="yes" active="yes"/>
+<layer number="43" name="vRestrict" color="2" fill="10" visible="yes" active="yes"/>
+<layer number="44" name="Drills" color="7" fill="1" visible="yes" active="yes"/>
+<layer number="45" name="Holes" color="7" fill="1" visible="yes" active="yes"/>
+<layer number="46" name="Milling" color="3" fill="1" visible="yes" active="yes"/>
+<layer number="47" name="Measures" color="7" fill="1" visible="yes" active="yes"/>
+<layer number="48" name="Document" color="7" fill="1" visible="yes" active="yes"/>
+<layer number="49" name="Reference" color="7" fill="1" visible="yes" active="yes"/>
+<layer number="51" name="tDocu" color="7" fill="1" visible="yes" active="yes"/>
+<layer number="52" name="bDocu" color="7" fill="1" visible="yes" active="yes"/>
 <layer number="88" name="SimResults" color="9" fill="1" visible="no" active="no"/>
 <layer number="89" name="SimProbes" color="9" fill="1" visible="no" active="no"/>
@@
 <board>
 <plain>
-<wire x1="0" y1="20.29289375" x2="0" y2="0.70710625" width="0" layer="20"/>
-<wire x1="0" y1="0.70710625" x2="0.70710625" y2="0" width="0" layer="20" curve="90"/>
-<wire x1="0.70710625" y1="0" x2="2" y2="0" width="0" layer="20"/>
-<wire x1="2" y1="0" x2="2" y2="-0.29289375" width="0" layer="20"/>
-<wire x1="2" y1="-0.29289375" x2="2.70710625" y2="-1" width="0" layer="20" curve="90"/>
-<wire x1="2.70710625" y1="-1" x2="11" y2="-1" width="0" layer="20"/>
-<wire x1="11" y1="-1" x2="12" y2="0" width="0" layer="20" curve="90"/>
-<wire x1="12" y1="0" x2="13.266159375" y2="0" width="0" layer="20"/>
-<wire x1="13.266159375" y1="0" x2="13.97" y2="0.635" width="0" layer="20" curve="89.756045"/>
-<wire x1="13.97" y1="0.635" x2="13.97" y2="20.32" width="0" layer="20"/>
-<wire x1="13.97" y1="20.32" x2="13.28985625" y2="21" width="0" layer="20" curve="90.245618"/>
-<wire x1="13.28985625" y1="21" x2="12" y2="21" width="0" layer="20"/>
-<wire x1="12" y1="21" x2="12" y2="21.29289375" width="0" layer="20"/>
-<wire x1="12" y1="21.29289375" x2="11.29289375" y2="22" width="0" layer="20" curve="90"/>
-<wire x1="11.29289375" y1="22" x2="2.70710625" y2="22" width="0" layer="20"/>
-<wire x1="2.70710625" y1="22" x2="2" y2="21.29289375" width="0" layer="20" curve="90"/>
-<wire x1="2" y1="21.29289375" x2="2" y2="21" width="0" layer="20"/>
-<wire x1="2" y1="21" x2="0.70710625" y2="21" width="0" layer="20"/>
-<wire x1="0.70710625" y1="21" x2="0" y2="20.29289375" width="0" layer="20" curve="90"/>
 <dimension x1="13.91" y1="0" x2="14" y2="21" x3="17.967784375" y3="10.4828" textsize="1.778" layer="47"/>
 <dimension x1="0" y1="0" x2="13.97" y2="0" x3="6.985" y3="-4" textsize="1.778" layer="47"/>
@@
 <text x="10.16" y="4.445" size="1.27" layer="25">R1</text>
 <text x="6.35" y="8.255" size="1.27" layer="25" rot="R90">150</text>
-<text x="6.35" y="12.7" size="1.27" layer="25" rot="R180">R2</text>
-<text x="12.7" y="12.065" size="0.6096" layer="25" rot="R270">optional-C</text>
+<text x="10.16" y="9.525" size="1.27" layer="25" rot="R90">R2</text>
+<text x="12.7" y="12.7" size="0.6096" layer="25" rot="R270">optional-C</text>
 <text x="8.255" y="18.415" size="1.27" layer="26" rot="MR270">C1</text>
 <text x="11.43" y="13.97" size="1.27" layer="26" rot="MR270">C2</text>
-<text x="8.255" y="19.685" size="1.27" layer="26" rot="MR180">10uF</text>
+<text x="6.92" y="19.785" size="1.27" layer="26" rot="MR180">10uF</text>
 <text x="6.35" y="15.24" size="1.27" layer="26" rot="MR180">100uF</text>
 <text x="12.7" y="10.16" size="1.27" layer="26" rot="MR0">AMS1117</text>
-<text x="6.35" y="6.35" size="1.27" layer="26" rot="MR180">AMS1117</text>
+<text x="7.62" y="6.985" size="1.27" layer="26" rot="MR180">1117</text>
 <text x="4.445" y="13.335" size="1.27" layer="26" rot="MR90">VCC</text>
 <text x="4.445" y="10.795" size="1.27" layer="26" rot="MR90">A</text>
 <text x="4.445" y="7.62" size="1.27" layer="26" rot="MR90">B</text>
 <text x="4.445" y="3.81" size="1.27" layer="26" rot="MR90">GND</text>
+<wire x1="0" y1="1.5" x2="2.1" y2="-0.6" width="0.001" layer="20" curve="-163.74"/>
+<wire x1="2.1" y1="-0.6" x2="11.9" y2="-0.6" width="0.001" layer="20"/>
+<wire x1="11.9" y1="-0.6" x2="14" y2="1.5" width="0.001" layer="20" curve="-163.74"/>
+<wire x1="14" y1="1.5" x2="14" y2="18.3" width="0.001" layer="20"/>
+<wire x1="14" y1="18.3" x2="11.9" y2="20.4" width="0.001" layer="20" curve="-163.74"/>
+<wire x1="11.9" y1="20.4" x2="2.1" y2="20.4" width="0.001" layer="20"/>
+<wire x1="2.1" y1="20.4" x2="0" y2="18.3" width="0.001" layer="20" curve="-163.74"/>
+<wire x1="0" y1="18.3" x2="0" y2="1.5" width="0.001" layer="20"/>
 </plain>
 <attributes>
@@
 <wire x1="7.43" y1="16.792209375" x2="8.147790625" y2="17.51" width="0.6096" layer="16"/>
 <contactref element="PAD4" pad="1"/>
-<via x="2.54" y="19.05" extent="1-16" drill="0.6" shape="square"/>
-<via x="3.81" y="19.05" extent="1-16" drill="0.6" shape="square"/>
-<via x="2.54" y="1.905" extent="1-16" drill="0.6" shape="square"/>
+<via x="2.84" y="17.75" extent="1-16" drill="0.6" shape="square"/>
+<via x="4.21" y="19.05" extent="1-16" drill="0.6" shape="square"/>
+<via x="2.64" y="2.305" extent="1-16" drill="0.6" shape="square"/>
 <via x="4.445" y="1.905" extent="1-16" drill="0.6" shape="square"/>
 <via x="6.35" y="1.905" extent="1-16" drill="0.6" shape="square"/>
-<wire x1="3.81" y1="19.05" x2="7.43" y2="16.792209375" width="0" layer="19" extent="16-16"/>
+<wire x1="4.21" y1="19.05" x2="2.84" y2="17.75" width="0" layer="19" extent="1-1"/>
+<wire x1="7.43" y1="16.792209375" x2="4.21" y2="19.05" width="0" layer="19" extent="16-16"/>
 </signal>
 <signal name="B">
