File: Water-Sensor/WaterSensor-V01-Build015.brd (EAGLE design)
At the start: 40 x 23 mm, 29 parts, among them IC1 LM358D, IC4 LM1117MPX-ADJ, T1 BC847, T2 BC847

Commit message: Water-Sensor V01
Parts:
- added TP1, TP2: TEST-POINT3, SparkFun-Connectors:PAD.03X.03
Connections:
- net SIG1: now also TP1.P$1
- net SIG2: now also TP2.P$1
Other:
- board text added: "10K"
- board text added: "10n"
- board text added: "10uF"
- board text added: "1K"
- board text added: "1Wire"
- board text added: "1Wire Dual-Rainsensor V0.1 www.neuby.de"
- board text added: "470"
- board text added: "470K"
- board text added: "AMS1117"
- board text added: "BC847"
- board text added: "C1"
- board text added: "C3"
- board text added: "C5"
- board text added: "C6 0.1u"
- board text added: "C7"
- board text added: "DS2413"
- board text added: "Fuse"
- board text added: "GND"
- board text added: "LM358"
- board text added: "R11"
- board text added: "R12 10K"
- board text added: "R13"
- board text added: "R2"
- board text added: "R3"
- board text added: "R5"
- board text added: "R6"
- board text added: "R7"
- board text added: "R8"
- board text added: "R9"
- board text added: "Sensor1"
- board text added: "Sensor2"
- board text added: "TP1"
- board text added: "TP2"
- board text added: "VCC"
- board text added: "VIN"
