File: Water-Sensor/WaterSensor-V01-Build015.sch (EAGLE design)
At the start: 29 parts, among them IC1 LM358D, IC4 LM1117MPX-ADJ, T1 BC847, T2 BC847

Commit message: Water-Sensor V01
Parts:
- added TP1, TP2: TEST-POINT3, SparkFun-Connectors:TEST-POINT3
Connections:
- net SIG1: now also TP1.1
- net SIG2: now also TP2.1
Other:
- note added: "OpAmp & 1Wire"
- note added: "Power"
Changed lines of the file:
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@@
 <part name="R13" library="rcl" library_urn="urn:adsk.eagle:library:334" deviceset="R-EU_" device="R0805W" package3d_urn="urn:adsk.eagle:package:23537/2" value="470K"/>
 <part name="T2" library="transistor" library_urn="urn:adsk.eagle:library:402" deviceset="BC847" device="" package3d_urn="urn:adsk.eagle:package:28738/2"/>
+<part name="TP1" library="SparkFun-Connectors" library_urn="urn:adsk.eagle:library:513" deviceset="TEST-POINT" device="3" package3d_urn="urn:adsk.eagle:package:38286/1"/>
+<part name="TP2" library="SparkFun-Connectors" library_urn="urn:adsk.eagle:library:513" deviceset="TEST-POINT" device="3" package3d_urn="urn:adsk.eagle:package:38286/1"/>
 </parts>
 <sheets>
 <sheet>
 <plain>
+<wire x1="99.06" y1="40.64" x2="241.3" y2="40.64" width="0.1524" layer="97"/>
+<wire x1="241.3" y1="40.64" x2="337.82" y2="40.64" width="0.1524" layer="97"/>
+<wire x1="337.82" y1="40.64" x2="337.82" y2="-139.7" width="0.1524" layer="97"/>
+<wire x1="337.82" y1="-139.7" x2="241.3" y2="-139.7" width="0.1524" layer="97"/>
+<wire x1="241.3" y1="-139.7" x2="99.06" y2="-139.7" width="0.1524" layer="97"/>
+<wire x1="99.06" y1="-139.7" x2="99.06" y2="40.64" width="0.1524" layer="97"/>
+<wire x1="241.3" y1="40.64" x2="241.3" y2="-139.7" width="0.1524" layer="97"/>
+<text x="246.38" y="33.02" size="5.08" layer="97">Power</text>
+<text x="101.6" y="33.02" size="5.08" layer="97">OpAmp &amp; 1Wire</text>
 </plain>
 <instances>
@@
 <attribute name="NAME" x="139.7" y="-96.52" size="1.778" layer="95"/>
 <attribute name="VALUE" x="139.7" y="-99.06" size="1.778" layer="96"/>
+</instance>
+<instance part="TP1" gate="G$1" x="132.08" y="17.78" smashed="yes" rot="R90">
+<attribute name="NAME" x="129.54" y="15.24" size="1.778" layer="95" font="vector" rot="R90"/>
+<attribute name="VALUE" x="134.62" y="15.24" size="1.778" layer="96" font="vector" rot="R90"/>
+</instance>
+<instance part="TP2" gate="G$1" x="132.08" y="-50.8" smashed="yes" rot="R90">
+<attribute name="NAME" x="129.54" y="-53.34" size="1.778" layer="95" font="vector" rot="R90"/>
+<attribute name="VALUE" x="134.62" y="-53.34" size="1.778" layer="96" font="vector" rot="R90"/>
 </instance>
 </instances>
@@
 <pinref part="LED2" gate="G$1" pin="C"/>
 <pinref part="U$1" gate="A" pin="IO"/>
-<wire x1="144.78" y1="-58.42" x2="129.54" y2="-58.42" width="0.1524" layer="91"/>
+<wire x1="144.78" y1="-58.42" x2="132.08" y2="-58.42" width="0.1524" layer="91"/>
+<pinref part="TP2" gate="G$1" pin="1"/>
+<wire x1="132.08" y1="-58.42" x2="129.54" y2="-58.42" width="0.1524" layer="91"/>
+<wire x1="132.08" y1="-50.8" x2="132.08" y2="-58.42" width="0.1524" layer="91"/>
+<junction x="132.08" y="-58.42"/>
 </segment>
 <segment>
@@
 <pinref part="LED1" gate="G$1" pin="C"/>
 <pinref part="U$1" gate="B" pin="IO"/>
-<wire x1="144.78" y1="12.7" x2="129.54" y2="12.7" width="0.1524" layer="91"/>
-</segment>
-<segment>
+<wire x1="144.78" y1="12.7" x2="132.08" y2="12.7" width="0.1524" layer="91"/>
+<pinref part="TP1" gate="G$1" pin="1"/>
+<wire x1="132.08" y1="12.7" x2="129.54" y2="12.7" width="0.1524" layer="91"/>
+<wire x1="132.08" y1="17.78" x2="132.08" y2="12.7" width="0.1524" layer="91"/>
+<junction x="132.08" y="12.7"/>
+</segment>
+<segment>
