File: I2C-Bus-Extender/P82B96-I2c-Bus-Extender-V02-005.brd (EAGLE design)
At the start: 32 x 16 mm, 15 parts

Commit message: I2C
Connections:
- net N$7 renamed RX-SDA
- net N$8 renamed TY-SCL
Other:
- board text added: "100n"
- board text added: "220p"
- board text added: "4K7"
- board text added: "750R"
- board text added: "BAT 54A"
- board text added: "I2C Extender V0.2"
- board text added: "P82B96"
- board text added: "R-SD"
- board text added: "SCL"
- board text added: "T-SC"
