File: I2C-Bus-Extender/P82B96-I2c-Bus-Extender-V02-005.sch (EAGLE design)
At the start: 15 parts

Commit message: I2C
Connections:
- net N$7 renamed RX-SDA
- net N$8 renamed TY-SCL
Changed lines of the file:
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@@
 <?xml version="1.0" encoding="utf-8"?>
 <!DOCTYPE eagle SYSTEM "eagle.dtd">
-<eagle version="9.3.0">
+<eagle version="9.1.1">
 <drawing>
 <settings>
@@
 </segment>
 </net>
-<net name="N$7" class="0">
+<net name="RX-SDA" class="0">
 <segment>
 <pinref part="CABLE" gate="G$1" pin="2"/>
@@
 </segment>
 </net>
-<net name="N$8" class="0">
+<net name="TY-SCL" class="0">
 <segment>
 <pinref part="CABLE" gate="G$1" pin="3"/>
