File: ESP8266-WLED/WeMos-WLED-V01-008.brd (EAGLE design)
At the start: 27 x 42 mm, 14 parts, among them J2 POWER_JACKPTH, U1 LDR, U2 DS18B20

Commit message: Cleanup Homematic
Connections:
- removed net 5V: JP4.8, JP8.8
- net +5V: now also JP4.8, JP8.8
Routing:
- net 5V: track 2.54 -> 0.00 mm
- net +5V: track 24.0 -> 26.6 mm
Changed lines of the file:
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@@
 <contactref element="JP7" pad="1"/>
-</signal>
-<signal name="5V" class="1">
-<contactref element="JP4" pad="8"/>
-<contactref element="JP8" pad="8"/>
-<wire x1="22.37" y1="27.21" x2="24.91" y2="27.21" width="0.9144" layer="16"/>
 </signal>
 <signal name="D4">
@@
 <wire x1="7.62" y1="10.16" x2="7.62" y2="11.43" width="0.9144" layer="16"/>
 <wire x1="7.62" y1="7.62" x2="7.62" y2="10.16" width="0.9144" layer="1"/>
+<contactref element="JP4" pad="8"/>
+<contactref element="JP8" pad="8"/>
+<wire x1="22.37" y1="27.21" x2="24.91" y2="27.21" width="0.9144" layer="16"/>
+<wire x1="14.1986" y1="20.32" x2="22.37" y2="27.21" width="0" layer="19" extent="16-16"/>
 </signal>
 <signal name="DQ">
