File: ESP8266-WLED/WeMos-WLED-V01-008.sch (EAGLE design)
At the start: 14 parts, among them J2 POWER_JACKPTH, U1 LDR, U2 DS18B20

Commit message: Cleanup Homematic
Connections:
- removed net 5V: JP4.8, JP8.8
- net +5V: now also JP4.8, JP8.8
Other:
- note added: "Historie: V02: Fix +5V at JP4+JP8"
Changed lines of the file:
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@@
 <text x="174.625" y="95.25" size="1.778" layer="94">D3/00</text>
 <text x="105.41" y="125.73" size="1.9304" layer="94" rot="R90" align="center">VIN DC</text>
+<text x="192.405" y="60.325" size="1.778" layer="97">Historie:
+V02: Fix +5V at JP4+JP8</text>
 </plain>
 <instances>
@@
 </segment>
 </net>
-<net name="5V" class="1">
-<segment>
-<pinref part="JP4" gate="G$1" pin="8"/>
-<label x="168.91" y="87.63" size="1.778" layer="95"/>
-<pinref part="JP8" gate="G$1" pin="8"/>
-<junction x="163.83" y="87.63"/>
-<wire x1="166.37" y1="87.63" x2="173.99" y2="87.63" width="0.1524" layer="91"/>
-<wire x1="163.83" y1="87.63" x2="166.37" y2="87.63" width="0.1524" layer="91"/>
-<junction x="166.37" y="87.63"/>
-</segment>
-</net>
 <net name="D4" class="0">
 <segment>
@@
 <junction x="145.415" y="128.905"/>
 </segment>
+<segment>
+<pinref part="JP4" gate="G$1" pin="8"/>
+<label x="168.91" y="87.63" size="1.778" layer="95"/>
+<pinref part="JP8" gate="G$1" pin="8"/>
+<junction x="163.83" y="87.63"/>
+<wire x1="166.37" y1="87.63" x2="179.705" y2="74.93" width="0.1524" layer="91"/>
+<wire x1="163.83" y1="87.63" x2="166.37" y2="87.63" width="0.1524" layer="91"/>
+<junction x="166.37" y="87.63"/>
+</segment>
 </net>
 <net name="DQ" class="0">
@@
 </drawing>
 <compatibility>
+<note version="6.3" minversion="6.2.2" severity="warning">
+Since Version 6.2.2 text objects can contain more than one line,
+which will not be processed correctly with this version.
+</note>
 <note version="8.2" severity="warning">
 Since Version 8.2, EAGLE supports online libraries. The ids
